File: hardware/circuits/base_station_pcb/base_station_pcb.kicad_sch (KiCad schematic)
At the start: 3 parts

Commit message: fix pcb and arduino nano pinout
Connections:
- net GND: now also Lora32.1 (GND); no longer Lora32.18 (GND)
- net UART_RX: now also Lora32.13 (GPIO2); no longer Lora32.6 (GPIO2)
- net VCC: now also Lora32.3 (3V3); no longer Lora32.16 (3V3)
Changed lines of the file:
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@@
 			)
+		)
+		(pin "18"
+		)
+		(pin "17"
+		)
+		(pin "16"
+		)
+		(pin "15"
+		)
+		(pin "14"
+		)
+		(pin "13"
+		)
+		(pin "12"
+		)
+		(pin "11"
+		)
+		(pin "10"
+		)
+		(pin "9"
+		)
+		(pin "8"
+		)
+		(pin "7"
+		)
+		(pin "6"
+		)
+		(pin "5"
+		)
+		(pin "4"
+		)
+		(pin "3"
+		)
+		(pin "2"
 		)
 		(pin "1"
 		)
-		(pin "2"
-		)
-		(pin "3"
-		)
-		(pin "4"
-		)
-		(pin "5"
-		)
-		(pin "6"
-		)
-		(pin "7"
-		)
-		(pin "8"
-		)
-		(pin "9"
-		)
-		(pin "10"
-		)
-		(pin "11"
-		)
-		(pin "12"
-		)
-		(pin "13"
-		)
-		(pin "14"
-		)
-		(pin "15"
-		)
-		(pin "16"
-		)
-		(pin "17"
-		)
-		(pin "18"
-		)
 		(pin "19"
