File: hardware/circuits/plane_pcb/plane_pcb.kicad_pcb (KiCad board)
At the start: 2 copper layers, 76.5 x 83.5 mm, 45 parts, among them J1 J1, J2 J2, J3 J3, J4 J4, U1 Magnetometer_Breakout, U2 U1

Commit message: fix pcb voltage divider
Parts:
- R16, R18, R20: value 47k -> 10k
- R17, R19, R21: value 10k -> 47k
Changed lines of the file:
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@@
 			)
 		)
-		(property "Value" "47k"
+		(property "Value" "10k"
 			(at 0 1.83 90)
 			(layer "F.Fab")
@@
 			)
 		)
-		(property "Value" "47k"
+		(property "Value" "10k"
 			(at 0 1.83 90)
 			(layer "F.Fab")
@@
 			)
 		)
-		(property "Value" "47k"
+		(property "Value" "10k"
 			(at 0 1.83 90)
 			(layer "F.Fab")
@@
 			)
 		)
-		(property "Value" "10k"
+		(property "Value" "47k"
 			(at 0 1.83 90)
 			(layer "F.Fab")
@@
 			)
 		)
-		(property "Value" "10k"
+		(property "Value" "47k"
 			(at 0 1.83 90)
 			(layer "F.Fab")
@@
 			)
 		)
-		(property "Value" "10k"
+		(property "Value" "47k"
 			(at 0 1.83 90)
 			(layer "F.Fab")
